File: kicad_files/power.kicad_sch (KiCad schematic)
At the start: 30 parts, among them J10 Battery Connector, U11 LT1963AxST-3.3, U12 TPS2121, U13 TPS54331DR

Commit message: update
Parts:
- removed U11: LT1963AxST-3.3, Package_TO_SOT_SMD:SOT-223-3_TabPin2, symbol Regulator_Linear:LT1963AxST-3.3
- added U14: AMS1117-3.3, Package_TO_SOT_SMD:SOT-223-3_TabPin2, symbol Regulator_Linear:AMS1117-3.3
Connections:
- net +3.3V_MAIN: now also U14.2 (VO)
- net +5V: now also U14.3 (VI)
- net GND: now also U14.1 (GND)
Changed lines of the file:
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@@
 	)
 	(junction
-		(at 50.8 73.66)
-		(diameter 0)
-		(color 0 0 0 0)
-	)
-	(junction
 		(at 82.55 154.94)
 		(diameter 0)
@@
 	)
 	(junction
+		(at 50.8 73.66)
+		(diameter 0)
+		(color 0 0 0 0)
+	)
+	(junction
 		(at 82.55 121.92)
 		(diameter 0)
@@
 	(wire
 		(pts
-			(xy 50.8 73.66) (xy 50.8 57.15)
-		)
-		(stroke
-			(width 0)
-			(type default)
-		)
-	)
-	(wire
-		(pts
 			(xy 48.26 57.15) (xy 50.8 57.15)
 		)
@@
 	(wire
 		(pts
-			(xy 50.8 73.66) (xy 50.8 90.17)
+			(xy 50.8 57.15) (xy 50.8 73.66)
 		)
 		(stroke
@@
 	(wire
 		(pts
-			(xy 40.64 57.15) (xy 40.64 63.5)
+			(xy 50.8 73.66) (xy 50.8 90.17)
 		)
 		(stroke
@@
 	(wire
 		(pts
-			(xy 40.64 83.82) (xy 40.64 90.17)
+			(xy 168.91 147.32) (xy 177.8 147.32)
 		)
 		(stroke
@@
 	(wire
 		(pts
-			(xy 168.91 147.32) (xy 177.8 147.32)
+			(xy 50.8 100.33) (xy 50.8 121.92)
 		)
 		(stroke
@@
 	(wire
 		(pts
-			(xy 50.8 100.33) (xy 50.8 121.92)
+			(xy 40.64 81.28) (xy 40.64 90.17)
+		)
+		(stroke
+			(width 0)
+			(type default)
+		)
+	)
+	(wire
+		(pts
+			(xy 40.64 57.15) (xy 40.64 66.04)
 		)
 		(stroke
@@
 	(wire
 		(pts
+			(xy 48.26 73.66) (xy 50.8 73.66)
+		)
+		(stroke
+			(width 0)
+			(type default)
+		)
+	)
+	(wire
+		(pts
 			(xy 50.8 57.15) (xy 50.8 46.99)
 		)
@@
 	)
 	(symbol
-		(lib_id "power:+5V")
-		(at 36.83 106.68 90)
+		(lib_id "Regulator_Linear:AMS1117-3.3")
+		(at 40.64 73.66 90)
 		(unit 1)
 		(body_style 1)
@@
 		(in_pos_files yes)
 		(dnp no)
-		(property "Reference" "#PWR081"
-			(at 40.64 106.68 0)
-			(hide yes)
+		(fields_autoplaced yes)
+		(property "Reference" "U14"
+			(at 36.83 72.3899 90)
 			(show_name no)
 			(do_not_autoplace no)
@@
 					(size 1.27 1.27)
 				)
+				(justify left)
 			)
 		)
-		(property "Value" "+5V"
-			(at 33.274 104.902 90)
+		(property "Value" "AMS1117-3.3"
+			(at 36.83 74.9299 90)
 			(show_name no)
 			(do_not_autoplace no)
@@
 					(size 1.27 1.27)
 				)
-				(justify right)
+				(justify left)
 			)
 		)
-		(property "Footprint" ""
-			(at 36.83 106.68 0)
+		(property "Footprint" "Package_TO_SOT_SMD:SOT-223-3_TabPin2"
+			(at 35.56 73.66 0)
 			(hide yes)
 			(show_name no)
@@
 			)
 		)
-		(property "Datasheet" ""
-			(at 36.83 106.68 0)
+		(property "Datasheet" "http://www.advanced-monolithic.com/pdf/ds1117.pdf"
+			(at 46.99 71.12 0)
 			(hide yes)
 			(show_name no)
@@
 			)
 		)
-		(property "Description" "Power symbol creates a global label with name \"+5V\""
-			(at 36.83 106.68 0)
+		(property "Description" "1A Low Dropout regulator, positive, 3.3V fixed output, SOT-223"
+			(at 40.64 73.66 0)
 			(hide yes)
 			(show_name no)
@@
 			)
 		)
+		(pin "3"
+		)
+		(pin "2"
+		)
 		(pin "1"
 		)
@@
 			(project "versorlite"
 				(path "/1a230af0-0a74-48f7-8607-b087121dda49/31c1824a-552d-4de4-ae9b-4526af07be04"
-					(reference "#PWR081")
+					(reference "U14")
 					(unit 1)
 				)
@@
 	)
 	(symbol
-		(lib_id "Device:C_Small")
-		(at 148.59 128.27 0)
+		(lib_id "power:+5V")
+		(at 36.83 106.68 90)
 		(unit 1)
 		(body_style 1)
@@
 		(in_pos_files yes)
 		(dnp no)
-		(fields_autoplaced yes)
-		(property "Reference" "C61"
-			(at 151.638 127.0062 0)
+		(property "Reference" "#PWR081"
+			(at 40.64 106.68 0)
+			(hide yes)
 			(show_name no)
 			(do_not_autoplace no)
@@
 					(size 1.27 1.27)
 				)
-				(justify left)
 			)
 		)
-		(property "Value" "10nf"
-			(at 151.638 129.5462 0)
+		(property "Value" "+5V"
+			(at 33.274 104.902 90)
 			(show_name no)
 			(do_not_autoplace no)
@@
 					(size 1.27 1.27)
 				)
-				(justify left)
+				(justify right)
 			)
 		)
-		(property "Footprint" "Capacitor_SMD:C_0402_1005Metric"
-			(at 148.59 128.27 0)
+		(property "Footprint" ""
+			(at 36.83 106.68 0)
 			(hide yes)
 			(show_name no)
@@
 		)
 		(property "Datasheet" ""
-			(at 148.59 128.27 0)
+			(at 36.83 106.68 0)
 			(hide yes)
 			(show_name no)
@@
 			)
 		)
-		(property "Description" "Unpolarized capacitor, small symbol"
-			(at 148.59 128.27 0)
+		(property "Description" "Power symbol creates a global label with name \"+5V\""
+			(at 36.83 106.68 0)
 			(hide yes)
 			(show_name no)
@@
 			)
 		)
-		(pin "2"
-		)
 		(pin "1"
 		)
@@
 			(project "versorlite"
 				(path "/1a230af0-0a74-48f7-8607-b087121dda49/31c1824a-552d-4de4-ae9b-4526af07be04"
-					(reference "C61")
+					(reference "#PWR081")
 					(unit 1)
 				)
@@
 	(symbol
 		(lib_id "Device:C_Small")
-		(at 45.72 100.33 90)
+		(at 148.59 128.27 0)
 		(unit 1)
 		(body_style 1)
@@
 		(dnp no)
 		(fields_autoplaced yes)
-		(property "Reference" "C53"
-			(at 45.7263 93.98 90)
+		(property "Reference" "C61"
+			(at 151.638 127.0062 0)
 			(show_name no)
 			(do_not_autoplace no)
@@
 					(size 1.27 1.27)
 				)
+				(justify left)
 			)
 		)
-		(property "Value" "10μf"
-			(at 45.7263 96.52 90)
+		(property "Value" "10nf"
+			(at 151.638 129.5462 0)
 			(show_name no)
 			(do_not_autoplace no)
@@
 					(size 1.27 1.27)
 				)
+				(justify left)
 			)
 		)
-		(property "Footprint" "Capacitor_SMD:C_0805_2012Metric"
-			(at 45.72 100.33 0)
+		(property "Footprint" "Capacitor_SMD:C_0402_1005Metric"
+			(at 148.59 128.27 0)
 			(hide yes)
 			(show_name no)
@@
 		)
 		(property "Datasheet" ""
-			(at 45.72 100.33 0)
+			(at 148.59 128.27 0)
 			(hide yes)
 			(show_name no)
@@
 		)
 		(property "Description" "Unpolarized capacitor, small symbol"
-			(at 45.72 100.33 0)
+			(at 148.59 128.27 0)
 			(hide yes)
 			(show_name no)
@@
 			)
 		)
-		(pin "1"
-		)
 		(pin "2"
 		)
+		(pin "1"
+		)
 		(instances
 			(project "versorlite"
 				(path "/1a230af0-0a74-48f7-8607-b087121dda49/31c1824a-552d-4de4-ae9b-4526af07be04"
-					(reference "C53")
+					(reference "C61")
 					(unit 1)
 				)
@@
 	)
 	(symbol
-		(lib_id "Regulator_Linear:LT1963AxST-3.3")
-		(at 43.18 73.66 90)
+		(lib_id "Device:C_Small")
+		(at 45.72 100.33 90)
 		(unit 1)
 		(body_style 1)
@@
 		(dnp no)
 		(fields_autoplaced yes)
-		(property "Reference" "U11"
-			(at 36.83 72.3899 90)
+		(property "Reference" "C53"
+			(at 45.7263 93.98 90)
 			(show_name no)
 			(do_not_autoplace no)
@@
 					(size 1.27 1.27)
 				)
-				(justify left)
 			)
 		)
-		(property "Value" "LT1963AxST-3.3"
-			(at 36.83 74.9299 90)
+		(property "Value" "10μf"
+			(at 45.7263 96.52 90)
 			(show_name no)
 			(do_not_autoplace no)
@@
 					(size 1.27 1.27)
 				)
-				(justify left)
 			)
 		)
-		(property "Footprint" "Package_TO_SOT_SMD:SOT-223-3_TabPin2"
-			(at 54.61 73.66 0)
+		(property "Footprint" "Capacitor_SMD:C_0805_2012Metric"
+			(at 45.72 100.33 0)
 			(hide yes)
 			(show_name no)
@@
 			)
 		)
-		(property "Datasheet" "https://www.analog.com/media/en/technical-documentation/data-sheets/1963aff.pdf"
-			(at 57.15 73.66 0)
+		(property "Datasheet" ""
+			(at 45.72 100.33 0)
 			(hide yes)
 			(show_name no)
@@
 			)
 		)
-		(property "Description" "3.3V, 1.5A, Low Noise, Fast Transient Response LDO Regulator, SOT-223"
-			(at 43.18 73.66 0)
+		(property "Description" "Unpolarized capacitor, small symbol"
+			(at 45.72 100.33 0)
 			(hide yes)
 			(show_name no)
@@
 			)
 		)
-		(pin "2"
-		)
-		(pin "3"
-		)
 		(pin "1"
 		)
+		(pin "2"
+		)
 		(instances
 			(project "versorlite"
 				(path "/1a230af0-0a74-48f7-8607-b087121dda49/31c1824a-552d-4de4-ae9b-4526af07be04"
-					(reference "U11")
+					(reference "C53")
 					(unit 1)
 				)

Commit message: final jlcpcb update
Parts:
- D6: value D_Schottky_Small -> Buckdiode
Changed lines of the file:
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@@
 		(fields_autoplaced yes)
 		(property "Reference" "D6"
-			(at 96.774 150.1139 90)
+			(at 96.52 150.1139 90)
 			(show_name no)
 			(do_not_autoplace no)
@@
 			)
 		)
-		(property "Value" "D_Schottky_Small"
-			(at 96.774 152.6539 90)
+		(property "Value" "Buckdiode"
+			(at 96.52 152.6539 90)
 			(show_name no)
 			(do_not_autoplace no)
